File: Arduino Telescope Interface/Telescope_Interface_shield.sch (EAGLE design)
At the start: 34 parts, among them IC1 40106N, IC2 24LC256P, J1 RJ45, J11 455-1750-1-ND, J12 455-1750-1-ND, J4 455-1750-1-ND, J8 455-1750-1-ND, J9 455-1750-1-ND, SW2 MOMENTARY-SWITCH-SPST-PTH-6.0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

Commit message: Motor driver calls added
Motor driver calls added and Diagnostics sketch expanded for motor and OLED testing
Parts:
- removed AL_A, AL_B, AZ_A, AZ_B: JUMPER-SMT_3_1-NC_TRACE_SILK, SparkFun-Jumpers:JUMPER-SMT_3_1-NC_TRACE_SILK
Connections:
- removed net N$1: AL_A.2, IC1A.O
- removed net N$14: AZ_A.2, IC1C.O
- removed net N$3: AL_B.2, IC1B.O
- removed net N$4: AZ_B.2, IC1D.O
- net AL_A: now also IC1B.O; no longer AL_A.1, AL_B.3
- net AL_B: now also IC1A.O; no longer AL_A.3, AL_B.1
- net AZ_A: now also IC1C.O; no longer AZ_A.3, AZ_B.1
- net AZ_B: now also IC1D.O; no longer AZ_A.1, AZ_B.3
Other:
- note added: "Encoder Direction Selection is now done in software"
- note added: "These Schmitt Triggers are used for noise immunity on the two most likely used Reference Sensors."
- note added: "XBee Header SAMD51 connections shown"
- note removed: "Encoder Direction Selection"
- note removed: "These Schmitt Triggers are used for noise immunity on the two Reference Sensors."
- note removed: "XBee Header M4 Metro connections shown"
Changed lines of the file:
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@@
 <part name="J12" library="SparkFun-Connectors" deviceset="CONN_03" device="" value="455-1750-1-ND"/>
 <part name="J13" library="SparkFun-Connectors" deviceset="CONN_04" device="PTH"/>
-<part name="AL_A" library="SparkFun-Jumpers" deviceset="JUMPER-SMT_3_1-NC_TRACE" device="_SILK" value=""/>
-<part name="AL_B" library="SparkFun-Jumpers" deviceset="JUMPER-SMT_3_1-NC_TRACE" device="_SILK" value=""/>
-<part name="AZ_A" library="SparkFun-Jumpers" deviceset="JUMPER-SMT_3_1-NC_TRACE" device="_SILK" value=""/>
-<part name="AZ_B" library="SparkFun-Jumpers" deviceset="JUMPER-SMT_3_1-NC_TRACE" device="_SILK" value=""/>
 <part name="J3" library="SparkFun-Connectors" deviceset="QWIIC_CONNECTOR" device="JS-1MM"/>
 <part name="JP1" library="SparkFun-Connectors" deviceset="M02" device="JST-PTH-2"/>
@@
 Level Shifter Header</text>
 <text x="43.18" y="60.96" size="1.778" layer="91">XBee Header
-M4 Metro connections
+SAMD51 connections
 shown</text>
 <text x="7.62" y="66.04" size="1.778" layer="91">QWIIC</text>
@@
 Do NOT attempt to use
 software with UNO.</text>
-<text x="175.26" y="63.5" size="1.778" layer="91">These Schmitt Triggers are used for noise immunity
-on the two Reference Sensors.</text>
-<text x="154.94" y="180.34" size="1.778" layer="91">Encoder Direction Selection</text>
+<text x="175.26" y="60.96" size="1.778" layer="91">These Schmitt Triggers are used for noise immunity
+on the two most likely used Reference Sensors.</text>
+<text x="157.48" y="177.8" size="1.778" layer="91">Encoder Direction Selection
+is now done in software</text>
 <text x="63.5" y="30.48" size="1.778" layer="91">5 volts regulated
 only on this
@@
 <attribute name="NAME" x="193.167" y="124.714" size="1.778" layer="95"/>
 </instance>
-<instance part="AL_A" gate="G$1" x="172.72" y="172.72" smashed="yes" rot="R180">
-<attribute name="NAME" x="170.18" y="172.339" size="1.778" layer="95" font="vector" rot="R180"/>
-<attribute name="VALUE" x="170.18" y="173.101" size="1.778" layer="96" font="vector" rot="R180" align="top-left"/>
-</instance>
-<instance part="AL_B" gate="G$1" x="172.72" y="160.02" smashed="yes" rot="R180">
-<attribute name="NAME" x="170.18" y="159.639" size="1.778" layer="95" font="vector" rot="R180"/>
-<attribute name="VALUE" x="170.18" y="160.401" size="1.778" layer="96" font="vector" rot="R180" align="top-left"/>
-</instance>
-<instance part="AZ_A" gate="G$1" x="172.72" y="147.32" smashed="yes" rot="R180">
-<attribute name="NAME" x="170.18" y="146.939" size="1.778" layer="95" font="vector" rot="R180"/>
-<attribute name="VALUE" x="170.18" y="147.701" size="1.778" layer="96" font="vector" rot="R180" align="top-left"/>
-</instance>
-<instance part="AZ_B" gate="G$1" x="172.72" y="134.62" smashed="yes" rot="R180">
-<attribute name="NAME" x="170.18" y="134.239" size="1.778" layer="95" font="vector" rot="R180"/>
-<attribute name="VALUE" x="170.18" y="135.001" size="1.778" layer="96" font="vector" rot="R180" align="top-left"/>
-</instance>
 <instance part="J3" gate="G$1" x="12.7" y="73.66" smashed="yes">
 <attribute name="VALUE" x="7.62" y="68.326" size="1.778" layer="96" font="vector" align="top-left"/>
@@
 </segment>
 </net>
-<net name="N$14" class="0">
-<segment>
-<pinref part="IC1" gate="C" pin="O"/>
-<pinref part="AZ_A" gate="G$1" pin="2"/>
-<wire x1="185.42" y1="147.32" x2="177.8" y2="147.32" width="0.1524" layer="91"/>
-</segment>
-</net>
 <net name="AL_B" class="0">
 <segment>
-<label x="160.02" y="177.8" size="1.27" layer="95" rot="MR0" xref="yes"/>
-<wire x1="162.56" y1="177.8" x2="160.02" y2="177.8" width="0.1524" layer="91"/>
-<wire x1="162.56" y1="177.8" x2="162.56" y2="154.94" width="0.1524" layer="91"/>
-<pinref part="AL_A" gate="G$1" pin="3"/>
-<wire x1="162.56" y1="177.8" x2="172.72" y2="177.8" width="0.1524" layer="91"/>
-<junction x="162.56" y="177.8"/>
-<pinref part="AL_B" gate="G$1" pin="1"/>
-<wire x1="162.56" y1="154.94" x2="172.72" y2="154.94" width="0.1524" layer="91"/>
+<label x="172.72" y="172.72" size="1.27" layer="95" rot="MR0" xref="yes"/>
+<wire x1="172.72" y1="172.72" x2="185.42" y2="172.72" width="0.1524" layer="91"/>
+<pinref part="IC1" gate="A" pin="O"/>
 </segment>
 <segment>
@@
 <net name="AL_A" class="0">
 <segment>
-<label x="160.02" y="167.64" size="1.27" layer="95" rot="MR0" xref="yes"/>
-<pinref part="AL_A" gate="G$1" pin="1"/>
-<wire x1="160.02" y1="167.64" x2="172.72" y2="167.64" width="0.1524" layer="91"/>
-<pinref part="AL_B" gate="G$1" pin="3"/>
-<wire x1="172.72" y1="167.64" x2="172.72" y2="165.1" width="0.1524" layer="91"/>
-<junction x="172.72" y="167.64"/>
+<label x="172.72" y="160.02" size="1.27" layer="95" rot="MR0" xref="yes"/>
+<wire x1="172.72" y1="160.02" x2="185.42" y2="160.02" width="0.1524" layer="91"/>
+<pinref part="IC1" gate="B" pin="O"/>
 </segment>
 <segment>
@@
 <net name="AZ_A" class="0">
 <segment>
-<label x="160.02" y="152.4" size="1.27" layer="95" rot="MR0" xref="yes"/>
-<wire x1="162.56" y1="152.4" x2="160.02" y2="152.4" width="0.1524" layer="91"/>
-<wire x1="162.56" y1="129.54" x2="162.56" y2="152.4" width="0.1524" layer="91"/>
-<pinref part="AZ_A" gate="G$1" pin="3"/>
-<wire x1="162.56" y1="152.4" x2="172.72" y2="152.4" width="0.1524" layer="91"/>
-<junction x="162.56" y="152.4"/>
-<pinref part="AZ_B" gate="G$1" pin="1"/>
-<wire x1="162.56" y1="129.54" x2="172.72" y2="129.54" width="0.1524" layer="91"/>
+<label x="172.72" y="147.32" size="1.27" layer="95" rot="MR0" xref="yes"/>
+<wire x1="172.72" y1="147.32" x2="185.42" y2="147.32" width="0.1524" layer="91"/>
+<pinref part="IC1" gate="C" pin="O"/>
 </segment>
 <segment>
@@
 <net name="AZ_B" class="0">
 <segment>
-<label x="160.02" y="142.24" size="1.27" layer="95" rot="MR0" xref="yes"/>
-<pinref part="AZ_A" gate="G$1" pin="1"/>
-<pinref part="AZ_B" gate="G$1" pin="3"/>
-<wire x1="172.72" y1="142.24" x2="172.72" y2="139.7" width="0.1524" layer="91"/>
-<wire x1="160.02" y1="142.24" x2="172.72" y2="142.24" width="0.1524" layer="91"/>
-<junction x="172.72" y="142.24"/>
+<label x="172.72" y="134.62" size="1.27" layer="95" rot="MR0" xref="yes"/>
+<wire x1="172.72" y1="134.62" x2="185.42" y2="134.62" width="0.1524" layer="91"/>
+<pinref part="IC1" gate="D" pin="O"/>
 </segment>
 <segment>
@@
 </segment>
 </net>
-<net name="N$1" class="0">
-<segment>
-<pinref part="IC1" gate="A" pin="O"/>
-<wire x1="177.8" y1="172.72" x2="185.42" y2="172.72" width="0.1524" layer="91"/>
-<pinref part="AL_A" gate="G$1" pin="2"/>
-</segment>
-</net>
-<net name="N$3" class="0">
-<segment>
-<pinref part="IC1" gate="B" pin="O"/>
-<wire x1="185.42" y1="160.02" x2="177.8" y2="160.02" width="0.1524" layer="91"/>
-<pinref part="AL_B" gate="G$1" pin="2"/>
-</segment>
-</net>
-<net name="N$4" class="0">
-<segment>
-<pinref part="IC1" gate="D" pin="O"/>
-<wire x1="185.42" y1="134.62" x2="177.8" y2="134.62" width="0.1524" layer="91"/>
-<pinref part="AZ_B" gate="G$1" pin="2"/>
-</segment>
-</net>

Commit message: Correction to interface shield
Correction to interface shield for Adafruit M4 Metro SAMD51 board that has 5V pin on ICSP connector
Connections:
- net 3.3V: no longer ICSP.2
- net 5V: now also ICSP.2
Other:
- note added: "Arduino Shield for Sparkfun SAMD51 Micro-Mod or Adafruit M4 Metro"
- note removed: "Arduino Shield for Sparkfun Redboard Turbo or Adafruit M4 Metro"
Changed lines of the file:
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@@
 <plain>
 <text x="40.64" y="175.26" size="2.032" layer="97" font="vector" ratio="15">Arduino Shield for
-Sparkfun Redboard Turbo
+Sparkfun SAMD51 Micro-Mod
 or Adafruit M4 Metro</text>
 <text x="40.64" y="121.92" size="1.651" layer="95" font="vector">Arduino_R3_Shield</text>
@@
 <label x="106.68" y="35.56" size="1.27" layer="95" xref="yes"/>
 </segment>
+<segment>
+<pinref part="ICSP" gate="G$1" pin="2"/>
+<wire x1="33.02" y1="114.3" x2="35.56" y2="114.3" width="0.1524" layer="91"/>
+<label x="35.56" y="114.3" size="1.27" layer="95" xref="yes"/>
+</segment>
 </net>
 <net name="MOSI" class="0">
@@
 </segment>
 <segment>
-<wire x1="33.02" y1="114.3" x2="35.56" y2="114.3" width="0.1524" layer="91"/>
-<pinref part="ICSP" gate="G$1" pin="2"/>
-<label x="35.56" y="114.3" size="1.27" layer="95" xref="yes"/>
-</segment>
-<segment>
